File: Hardware/Hinge Tester/Hinge Tester.sch (KiCad schematic (older format))
At the start: 5 parts

Commit message: Add terminal block footprints
Parts:
- J? (x2): footprint (none) -> TerminalBlock_TE-Connectivity:TerminalBlock_TE_282834-2_1x02_P2.54mm_Horizontal
- J?: footprint (none) -> TerminalBlock_RND:TerminalBlock_RND_205-00234_1x04_P5.08mm_Horizontal
Changed lines of the file:
@@
-$Comp
-L Connector:Conn_01x02_Female J?
-U 1 1 6361E597
-P 4400 1700
-F 0 "J?" H 4428 1676 50  0000 L CNN
-F 1 "Conn_01x02_Female" H 4428 1585 50  0000 L CNN
-F 2 "" H 4400 1700 50  0001 C CNN
-F 3 "~" H 4400 1700 50  0001 C CNN
-	1    4400 1700
-	1    0    0    -1
-$EndComp
 $Comp
 L Connector:Conn_01x02_Female J?
@@
 F 0 "J?" H 6028 1676 50  0000 L CNN
 F 1 "Conn_01x02_Female" H 6028 1585 50  0000 L CNN
-F 2 "" H 6000 1700 50  0001 C CNN
+F 2 "TerminalBlock_TE-Connectivity:TerminalBlock_TE_282834-2_1x02_P2.54mm_Horizontal" H 6000 1700 50  0001 C CNN
 F 3 "~" H 6000 1700 50  0001 C CNN
 	1    6000 1700
@@
 F 0 "J?" H 2678 4076 50  0000 L CNN
 F 1 "Conn_01x04_Female" H 2678 3985 50  0000 L CNN
-F 2 "" H 2650 4100 50  0001 C CNN
+F 2 "TerminalBlock_RND:TerminalBlock_RND_205-00234_1x04_P5.08mm_Horizontal" H 2650 4100 50  0001 C CNN
 F 3 "~" H 2650 4100 50  0001 C CNN
 	1    2650 4100
@@
 Wire Wire Line
 	8100 4350 8000 4350
+$Comp
+L Connector:Conn_01x02_Female J?
+U 1 1 6361E597
+P 4400 1700
+F 0 "J?" H 4428 1676 50  0000 L CNN
+F 1 "Conn_01x02_Female" H 4428 1585 50  0000 L CNN
+F 2 "TerminalBlock_TE-Connectivity:TerminalBlock_TE_282834-2_1x02_P2.54mm_Horizontal" H 4400 1700 50  0001 C CNN
+F 3 "~" H 4400 1700 50  0001 C CNN
+	1    4400 1700
+	1    0    0    -1
+$EndComp
 $EndSCHEMATC

Commit message: Add rough board layout
Parts:
- removed U?: Adafruit_ItsyBitsy_M4_Express, symbol Breakouts:Adafruit_ItsyBitsy_M4_Express
- added U?: Adafruit_ItsyBitsy_M4_Express, symbol Breakouts:Adafruit_ItsyBitsy_M4_Express
- U1: renamed from U?; footprint (none) -> Modules:TB67S128FTG
- gave numbers to parts that had none: 3
Connections:
- net +3V3: now also U?.2 (3V3)
- net +5V: now also U?.33 (VBAT)
- net DIR: now also U?.29 (D12)
- net EN: now also U?.28 (D11)
- net GND: now also U?.32 (GND)
- net M0: now also U?.25 (D7)
- net M1: now also U?.26 (D9)
- net M2: now also U?.27 (D10)
- net STEP: now also U?.30 (D13)
Changed lines of the file:
@@
 $EndDescr
 $Comp
-L power:+5V #PWR?
+L power:+5V #PWR0101
 U 1 1 6361D18B
 P 5700 1600
-F 0 "#PWR?" H 5700 1450 50  0001 C CNN
+F 0 "#PWR0101" H 5700 1450 50  0001 C CNN
 F 1 "+5V" H 5715 1773 50  0000 C CNN
 F 2 "" H 5700 1600 50  0001 C CNN
@@
 $EndComp
 $Comp
-L power:+24V #PWR?
+L power:+24V #PWR0102
 U 1 1 6361D49F
 P 2750 4550
-F 0 "#PWR?" H 2750 4400 50  0001 C CNN
+F 0 "#PWR0102" H 2750 4400 50  0001 C CNN
 F 1 "+24V" H 2765 4723 50  0000 C CNN
 F 2 "" H 2750 4550 50  0001 C CNN
@@
 $EndComp
 $Comp
-L power:GND #PWR?
+L power:GND #PWR0103
 U 1 1 6361DBF4
 P 8250 3650
-F 0 "#PWR?" H 8250 3400 50  0001 C CNN
+F 0 "#PWR0103" H 8250 3400 50  0001 C CNN
 F 1 "GND" H 8255 3477 50  0000 C CNN
 F 2 "" H 8250 3650 50  0001 C CNN
@@
 $EndComp
 $Comp
-L Connector:Conn_01x02_Female J?
+L Connector:Conn_01x02_Female J3
 U 1 1 6361FE6E
 P 6000 1700
-F 0 "J?" H 6028 1676 50  0000 L CNN
+F 0 "J3" H 6028 1676 50  0000 L CNN
 F 1 "Conn_01x02_Female" H 6028 1585 50  0000 L CNN
 F 2 "TerminalBlock_TE-Connectivity:TerminalBlock_TE_282834-2_1x02_P2.54mm_Horizontal" H 6000 1700 50  0001 C CNN
@@
 $EndComp
 $Comp
-L Connector:Conn_01x04_Female J?
+L Connector:Conn_01x04_Female J1
 U 1 1 6362003C
 P 2650 4100
-F 0 "J?" H 2678 4076 50  0000 L CNN
+F 0 "J1" H 2678 4076 50  0000 L CNN
 F 1 "Conn_01x04_Female" H 2678 3985 50  0000 L CNN
 F 2 "TerminalBlock_RND:TerminalBlock_RND_205-00234_1x04_P5.08mm_Horizontal" H 2650 4100 50  0001 C CNN
@@
 $EndComp
 $Comp
-L Breakouts:Adafruit_ItsyBitsy_M4_Express U?
-U 1 1 63620E23
-P 7550 3450
-F 0 "U?" H 7550 3615 50  0000 C CNN
-F 1 "Adafruit_ItsyBitsy_M4_Express" H 7550 3524 50  0000 C CNN
-F 2 "" H 7550 3650 50  0001 C CNN
-F 3 "" H 7550 3650 50  0001 C CNN
-	1    7550 3450
-	1    0    0    -1
-$EndComp
-$Comp
-L Breakouts:TB67S128FTG U?
+L Breakouts:TB67S128FTG U1
 U 1 1 63628E93
 P 3700 2900
-F 0 "U?" H 3675 361 50  0000 C CNN
+F 0 "U1" H 3675 361 50  0000 C CNN
 F 1 "TB67S128FTG" H 3675 270 50  0000 C CNN
-F 2 "" H 3700 2950 50  0001 C CNN
+F 2 "Modules:TB67S128FTG" H 3700 2950 50  0001 C CNN
 F 3 "" H 3700 2950 50  0001 C CNN
 	1    3700 2900
@@
 $EndComp
 $Comp
-L power:+24V #PWR?
+L power:+24V #PWR0104
 U 1 1 6362E7A2
 P 4100 1600
-F 0 "#PWR?" H 4100 1450 50  0001 C CNN
+F 0 "#PWR0104" H 4100 1450 50  0001 C CNN
 F 1 "+24V" H 4115 1773 50  0000 C CNN
 F 2 "" H 4100 1600 50  0001 C CNN
@@
 $EndComp
 $Comp
-L power:GND #PWR?
+L power:GND #PWR0105
 U 1 1 6362F794
 P 2850 4350
-F 0 "#PWR?" H 2850 4100 50  0001 C CNN
+F 0 "#PWR0105" H 2850 4100 50  0001 C CNN
 F 1 "GND" H 2855 4177 50  0000 C CNN
 F 2 "" H 2850 4350 50  0001 C CNN
@@
 $EndComp
 $Comp
-L power:GND #PWR?
+L power:GND #PWR0106
 U 1 1 63630014
 P 4500 4900
-F 0 "#PWR?" H 4500 4650 50  0001 C CNN
+F 0 "#PWR0106" H 4500 4650 50  0001 C CNN
 F 1 "GND" H 4505 4727 50  0000 C CNN
 F 2 "" H 4500 4900 50  0001 C CNN
@@
 $EndComp
 $Comp
-L power:GND #PWR?
+L power:GND #PWR0107
 U 1 1 63630C1A
 P 4100 1900
-F 0 "#PWR?" H 4100 1650 50  0001 C CNN
+F 0 "#PWR0107" H 4100 1650 50  0001 C CNN
 F 1 "GND" H 4105 1727 50  0000 C CNN
 F 2 "" H 4100 1900 50  0001 C CNN
@@
 	5700 1800 5700 1900
 $Comp
-L power:+5V #PWR?
+L power:+5V #PWR0108
 U 1 1 63641C56
 P 8250 3450
-F 0 "#PWR?" H 8250 3300 50  0001 C CNN
+F 0 "#PWR0108" H 8250 3300 50  0001 C CNN
 F 1 "+5V" H 8265 3623 50  0000 C CNN
 F 2 "" H 8250 3450 50  0001 C CNN
@@
 $EndComp
 $Comp
-L power:GND #PWR?
+L power:GND #PWR0109
 U 1 1 63643310
 P 5700 1900
-F 0 "#PWR?" H 5700 1650 50  0001 C CNN
+F 0 "#PWR0109" H 5700 1650 50  0001 C CNN
 F 1 "GND" H 5705 1727 50  0000 C CNN
 F 2 "" H 5700 1900 50  0001 C CNN
@@
 	4500 4700 4400 4700
 $Comp
-L power:+3.3V #PWR?
+L power:+3.3V #PWR0110
 U 1 1 636469AA
 P 6800 3450
-F 0 "#PWR?" H 6800 3300 50  0001 C CNN
+F 0 "#PWR0110" H 6800 3300 50  0001 C CNN
 F 1 "+3.3V" H 6815 3623 50  0000 C CNN
 F 2 "" H 6800 3450 50  0001 C CNN
@@
 $EndComp
 $Comp
-L power:+3.3V #PWR?
+L power:+3.3V #PWR0111
 U 1 1 63647E6F
 P 4700 5000
-F 0 "#PWR?" H 4700 4850 50  0001 C CNN
+F 0 "#PWR0111" H 4700 4850 50  0001 C CNN
 F 1 "+3.3V" H 4715 5173 50  0000 C CNN
 F 2 "" H 4700 5000 50  0001 C CNN
@@
 	8100 4350 8000 4350
 $Comp
-L Connector:Conn_01x02_Female J?
+L Connector:Conn_01x02_Female J2
 U 1 1 6361E597
 P 4400 1700
-F 0 "J?" H 4428 1676 50  0000 L CNN
+F 0 "J2" H 4428 1676 50  0000 L CNN
 F 1 "Conn_01x02_Female" H 4428 1585 50  0000 L CNN
 F 2 "TerminalBlock_TE-Connectivity:TerminalBlock_TE_282834-2_1x02_P2.54mm_Horizontal" H 4400 1700 50  0001 C CNN
@@
 	1    0    0    -1
 $EndComp
+$Comp
+L Breakouts:Adafruit_ItsyBitsy_M4_Express U?
+U 1 1 63624B99
+P 7550 3450
+F 0 "U?" H 7550 3615 50  0000 C CNN
+F 1 "Adafruit_ItsyBitsy_M4_Express" H 7550 3524 50  0000 C CNN
+F 2 "" H 7550 3650 50  0001 C CNN
+F 3 "" H 7550 3650 50  0001 C CNN
+	1    7550 3450
+	1    0    0    -1
+$EndComp
