File: Hardware/Hinge Tester/Hinge Tester.kicad_pcb (KiCad board)
At the start: 2 copper layers, 76.2 x 50.8 mm, 5 parts, among them J1 Conn_01x04_Female, J2 Conn_01x02_Female, J3 Conn_01x02_Female, U1 TB67S128FTG, U2 Adafruit_ItsyBitsy_M4_Express

Commit message: Improve page layout
Parts:
- moved J2 9.25 mm to (130.8, 81.3)
- moved J3 9.25 mm to (120.7, 81.3)
- moved U1 9.25 mm to (153.7, 104.1)
- moved U2 9.25 mm to (171.4, 101.6)
- moved J1 9.25 mm to (141.0, 81.3)
Routing:
- net +5V: track 0.00 -> 85.3 mm
- net +3V3: track 0.00 -> 61.6 mm
- net M0: track 0.00 -> 44.0 mm
- net M1: track 0.00 -> 40.4 mm
- net M2: track 0.00 -> 36.8 mm
- net DIR: track 0.00 -> 33.1 mm
- net STEP: track 0.00 -> 29.6 mm
- net EN: track 0.00 -> 28.1 mm
Changed lines of the file:
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@@
     (thickness 1.6)
     (drawings 8)
-    (tracks 10)
+    (tracks 37)
     (zones 0)
     (modules 5)
     (nets 57)
   )
-  (page A4)
+  (page USLetter)
+  (title_block
+    (title "Hinge Tester")
+    (rev 0.1.0)
+    (company MobileDemand)
+  )
   (layers
     (0 F.Cu signal)
@@
   )
   (setup
-    (last_trace_width 1.5)
+    (last_trace_width 0.75)
+    (user_trace_width 0.75)
     (user_trace_width 1.5)
     (trace_clearance 0.2)
@@
   )
   (module TerminalBlock_RND:TerminalBlock_RND_205-00234_1x04_P5.08mm_Horizontal (layer F.Cu)
-    (at 132.08 83.82)
+    (at 140.97 81.28)
     (descr "terminal block RND 205-00234, 4 pins, pitch 5.08mm, size 20.3x8.45mm^2, drill diamater 1.1mm, pad diameter 2.1mm, see http://cdn-reichelt.de/documents/datenblatt/C151/RND_205-00232_DB_EN.pdf, script-generated using https://github.com/pointhi/kicad-footprint-generator/scripts/TerminalBlock_RND")
     (tags "THT terminal block RND 205-00234 pitch 5.08mm size 20.3x8.45mm^2 drill 1.1mm pad 2.1mm")
@@
   )
   (module TerminalBlock_TE-Connectivity:TerminalBlock_TE_282834-2_1x02_P2.54mm_Horizontal (layer F.Cu)
-    (at 121.92 83.82)
+    (at 130.81 81.28)
     (descr "Terminal Block TE 282834-2, 2 pins, pitch 2.54mm, size 5.54x6.5mm^2, drill diamater 1.1mm, pad diameter 2.1mm, see http://www.te.com/commerce/DocumentDelivery/DDEController?Action=showdoc&DocId=Customer+Drawing%7F282834%7FC1%7Fpdf%7FEnglish%7FENG_CD_282834_C1.pdf, script-generated using https://github.com/pointhi/kicad-footprint-generator/scripts/TerminalBlock_TE-Connectivity")
     (tags "THT Terminal Block TE 282834-2 pitch 2.54mm size 5.54x6.5mm^2 drill 1.1mm pad 2.1mm")
@@
   )
   (module TerminalBlock_TE-Connectivity:TerminalBlock_TE_282834-2_1x02_P2.54mm_Horizontal (layer F.Cu)
-    (at 111.76 83.82)
+    (at 120.65 81.28)
     (descr "Terminal Block TE 282834-2, 2 pins, pitch 2.54mm, size 5.54x6.5mm^2, drill diamater 1.1mm, pad diameter 2.1mm, see http://www.te.com/commerce/DocumentDelivery/DDEController?Action=showdoc&DocId=Customer+Drawing%7F282834%7FC1%7Fpdf%7FEnglish%7FENG_CD_282834_C1.pdf, script-generated using https://github.com/pointhi/kicad-footprint-generator/scripts/TerminalBlock_TE-Connectivity")
     (tags "THT Terminal Block TE 282834-2 pitch 2.54mm size 5.54x6.5mm^2 drill 1.1mm pad 2.1mm")
@@
   )
   (module Modules:TB67S128FTG (layer F.Cu)
-    (at 144.78 106.68 270)
+    (at 153.67 104.14 270)
     (fp_text reference U1 (at 0 17.01 90) (layer F.SilkS)
       (effects (font (size 1 1) (thickness 0.15)))
@@
   )
   (module Modules:Adafruit_ItsyBitsy_M4 (layer F.Cu)
-    (at 162.56 104.14 180)
+    (at 171.45 101.6 180)
     (fp_text reference U2 (at 0 0.5) (layer F.SilkS)
       (effects (font (size 1 1) (thickness 0.15)))
@@
       (net 7 +5V))
   )
-  (gr_arc (start 104.14 124.46) (end 101.6 124.46) (angle -90) (layer Edge.Cuts) (width 0.05))
-  (gr_arc (start 175.26 124.46) (end 175.26 127) (angle -90) (layer Edge.Cuts) (width 0.05))
-  (gr_arc (start 104.14 78.74) (end 104.14 76.2) (angle -90) (layer Edge.Cuts) (width 0.05))
-  (gr_arc (start 175.26 78.74) (end 177.8 78.74) (angle -90) (layer Edge.Cuts) (width 0.05))
-  (gr_line (start 177.8 78.74) (end 177.8 124.46) (layer Edge.Cuts) (width 0.05))
-  (gr_line (start 104.14 76.2) (end 175.26 76.2) (layer Edge.Cuts) (width 0.05))
-  (gr_line (start 101.6 124.46) (end 101.6 78.74) (layer Edge.Cuts) (width 0.05))
-  (gr_line (start 175.26 127) (end 104.14 127) (layer Edge.Cuts) (width 0.05))
-  (segment (start 129.54 86.36) (end 132.08 83.82) (width 1.5) (layer B.Cu) (net 1))
-  (segment (start 129.54 92.71) (end 129.54 86.36) (width 1.5) (layer B.Cu) (net 1))
-  (segment (start 132.08 88.9) (end 137.16 83.82) (width 1.5) (layer B.Cu) (net 2))
-  (segment (start 132.08 92.71) (end 132.08 88.9) (width 1.5) (layer B.Cu) (net 2))
-  (segment (start 134.62 91.44) (end 142.24 83.82) (width 1.5) (layer B.Cu) (net 3))
-  (segment (start 134.62 92.71) (end 134.62 91.44) (width 1.5) (layer B.Cu) (net 3))
-  (segment (start 138.43 92.71) (end 147.32 83.82) (width 1.5) (layer B.Cu) (net 4))
-  (segment (start 137.16 92.71) (end 138.43 92.71) (width 1.5) (layer B.Cu) (net 4))
-  (segment (start 119.38 92.71) (end 121.92 92.71) (width 1.5) (layer B.Cu) (net 6))
-  (segment (start 121.92 92.71) (end 121.92 83.82) (width 1.5) (layer B.Cu) (net 6))
+  (gr_arc (start 113.03 121.92) (end 110.49 121.92) (angle -90) (layer Edge.Cuts) (width 0.05))
+  (gr_arc (start 184.15 121.92) (end 184.15 124.46) (angle -90) (layer Edge.Cuts) (width 0.05))
+  (gr_arc (start 113.03 76.2) (end 113.03 73.66) (angle -90) (layer Edge.Cuts) (width 0.05))
+  (gr_arc (start 184.15 76.2) (end 186.69 76.2) (angle -90) (layer Edge.Cuts) (width 0.05))
+  (gr_line (start 186.69 76.2) (end 186.69 121.92) (layer Edge.Cuts) (width 0.05))
+  (gr_line (start 113.03 73.66) (end 184.15 73.66) (layer Edge.Cuts) (width 0.05))
+  (gr_line (start 110.49 121.92) (end 110.49 76.2) (layer Edge.Cuts) (width 0.05))
+  (gr_line (start 184.15 124.46) (end 113.03 124.46) (layer Edge.Cuts) (width 0.05))
+  (segment (start 138.43 83.82) (end 140.97 81.28) (width 1.5) (layer B.Cu) (net 1))
+  (segment (start 138.43 90.17) (end 138.43 83.82) (width 1.5) (layer B.Cu) (net 1))
+  (segment (start 140.97 86.36) (end 146.05 81.28) (width 1.5) (layer B.Cu) (net 2))
+  (segment (start 140.97 90.17) (end 140.97 86.36) (width 1.5) (layer B.Cu) (net 2))
+  (segment (start 143.51 88.9) (end 151.13 81.28) (width 1.5) (layer B.Cu) (net 3))
+  (segment (start 143.51 90.17) (end 143.51 88.9) (width 1.5) (layer B.Cu) (net 3))
+  (segment (start 147.32 90.17) (end 156.21 81.28) (width 1.5) (layer B.Cu) (net 4))
+  (segment (start 146.05 90.17) (end 147.32 90.17) (width 1.5) (layer B.Cu) (net 4))
+  (segment (start 128.27 90.17) (end 130.81 90.17) (width 1.5) (layer B.Cu) (net 6))
+  (segment (start 130.81 90.17) (end 130.81 81.28) (width 1.5) (layer B.Cu) (net 6))
+  (segment (start 166.37 115.57) (end 163.83 118.11) (width 0.75) (layer B.Cu) (net 7))
+  (segment (start 166.37 83.82) (end 166.37 115.57) (width 0.75) (layer B.Cu) (net 7))
+  (segment (start 160.02 77.47) (end 166.37 83.82) (width 0.75) (layer B.Cu) (net 7))
+  (segment (start 124.46 77.47) (end 160.02 77.47) (width 0.75) (layer B.Cu) (net 7))
+  (segment (start 120.65 81.28) (end 124.46 77.47) (width 0.75) (layer B.Cu) (net 7))
+  (segment (start 173.99 120.65) (end 179.07 115.57) (width 0.25) (layer B.Cu) (net 9))
+  (segment (start 123.19 120.65) (end 173.99 120.65) (width 0.25) (layer B.Cu) (net 9))
+  (segment (start 120.65 118.11) (end 123.19 120.65) (width 0.25) (layer B.Cu) (net 9))
+  (segment (start 157.335001 104.284999) (end 163.83 97.79) (width 0.25) (layer B.Cu) (net 27))
+  (segment (start 142.095001 104.284999) (end 157.335001 104.284999) (width 0.25) (layer B.Cu) (net 27))
+  (segment (start 128.27 118.11) (end 142.095001 104.284999) (width 0.25) (layer B.Cu) (net 27))
+  (segment (start 142.384999 106.535001) (end 130.81 118.11) (width 0.25) (layer B.Cu) (net 28))
+  (segment (start 157.624999 106.535001) (end 142.384999 106.535001) (width 0.25) (layer B.Cu) (net 28))
+  (segment (start 163.83 100.33) (end 157.624999 106.535001) (width 0.25) (layer B.Cu) (net 28))
+  (segment (start 157.624999 109.075001) (end 142.384999 109.075001) (width 0.25) (layer B.Cu) (net 29))
+  (segment (start 142.384999 109.075001) (end 133.35 118.11) (width 0.25) (layer B.Cu) (net 29))
+  (segment (start 163.83 102.87) (end 157.624999 109.075001) (width 0.25) (layer B.Cu) (net 29))
+  (segment (start 150.004999 111.615001) (end 143.51 118.11) (width 0.25) (layer B.Cu) (net 30))
+  (segment (start 157.624999 111.615001) (end 150.004999 111.615001) (width 0.25) (layer B.Cu) (net 30))
+  (segment (start 163.83 105.41) (end 157.624999 111.615001) (width 0.25) (layer B.Cu) (net 30))
+  (segment (start 140.97 118.11) (end 143.51 118.11) (width 0.25) (layer B.Cu) (net 30))
+  (segment (start 138.43 118.11) (end 147.32 109.22) (width 0.25) (layer F.Cu) (net 44))
+  (segment (start 162.56 109.22) (end 163.83 110.49) (width 0.25) (layer F.Cu) (net 44))
+  (segment (start 147.32 109.22) (end 162.56 109.22) (width 0.25) (layer F.Cu) (net 44))
+  (segment (start 147.175001 106.824999) (end 135.89 118.11) (width 0.25) (layer F.Cu) (net 45))
+  (segment (start 162.704999 106.824999) (end 147.175001 106.824999) (width 0.25) (layer F.Cu) (net 45))
+  (segment (start 163.83 107.95) (end 162.704999 106.824999) (width 0.25) (layer F.Cu) (net 45))
   (zone (net 5) (net_name GND) (layer F.Cu) (hatch edge 0.508)
     (connect_pads (clearance 0.508))
     (min_thickness 0.254)
-    (fill (arc_segments 32) (thermal_gap 0.508) (thermal_bridge_width 0.508))
+    (fill yes (arc_segments 32) (thermal_gap 0.508) (thermal_bridge_width 0.508))
     (polygon
       (pts
-        (xy 180.34 129.54) (xy 99.06 129.54) (xy 99.06 73.66) (xy 180.34 73.66)
+        (xy 189.23 127) (xy 107.95 127) (xy 107.95 71.12) (xy 189.23 71.12)
       )
     )
@@
     (connect_pads (clearance 0.508))
     (min_thickness 0.254)
-    (fill (arc_segments 32) (thermal_gap 0.508) (thermal_bridge_width 0.508))
+    (fill yes (arc_segments 32) (thermal_gap 0.508) (thermal_bridge_width 0.508))
     (polygon
       (pts
-        (xy 180.34 129.54) (xy 99.06 129.54) (xy 99.06 73.66) (xy 180.34 73.66)
+        (xy 189.23 127) (xy 107.95 127) (xy 107.95 71.12) (xy 189.23 71.12)
       )
     )
